Commit message: It's dirty to change the URDF here, but easy for now...

File: kortex_description/robots/kortex_robot.xacro (robot description, xacro)
@@ -36,7 +36,21 @@
         <!-- If no gripper, define tool frame here -->
         <xacro:if value="${not gripper}">
-            <link name="${prefix}tool_frame"/>
+            <link name="${prefix}tool_frame">
+              <visual>
+                <origin xyz="0 0 0" rpy="0 0 0" />
+                <geometry>
+                  <mesh filename="package://weedbot_description/meshes/rosebud.dae" />
+                </geometry>
+              </visual>
+              <collision>
+                <origin xyz="0 0 0" rpy="0 0 0" />
+                <geometry>
+                  <mesh filename="package://weedbot_description/meshes/rosebud.dae" />
+                </geometry>
+              </collision>
+            </link>
             <joint name="${prefix}tool_frame_joint" type="fixed">
-                <origin xyz="0 0 0" rpy="0 0 0" />
+                <!-- origin xyz="0 0 0" rpy="0 0 0" / -->
+                <origin xyz="-0.41 0 0.02" rpy="0 -1.5707 3.14159" />
                 <parent link="${prefix}${last_arm_link}" />
                 <child link="${prefix}tool_frame" />
