Commit message: more dirty little updates to the urdf

File: kortex_description/arms/gen3/7dof/urdf/gen3_macro.xacro (robot description, xacro)
@@ -50,5 +50,5 @@
     <joint
       name="${prefix}joint_1"
-      type="continuous">
+      type="revolute">
       <origin xyz="0 0 0.15643" rpy="3.1416 2.7629E-18 -4.9305E-36" />
       <parent
@@ -58,7 +58,5 @@
       <axis
         xyz="0 0 1" />
-      <limit
-        effort="39"
-        velocity="1.3963" />
+      <limit lower="-2.41" upper="2.41" effort="39" velocity="0.87" />
     </joint>
     <link name="${prefix}half_arm_1_link">
@@ -94,5 +92,5 @@
       <axis
         xyz="0 0 1" />
-      <limit lower="-2.41" upper="2.41" effort="39" velocity="1.3963" />
+      <limit lower="-2.41" upper="2.41" effort="39" velocity="0.87" />
     </joint>
     <link name="${prefix}half_arm_2_link">
@@ -120,5 +118,5 @@
     <joint
       name="${prefix}joint_3"
-      type="continuous">
+      type="revolute">
       <origin xyz="0 -0.21038 -0.006375" rpy="-1.5708 1.2326E-32 -2.9122E-16" />
       <parent
@@ -128,7 +126,5 @@
       <axis
         xyz="0 0 1" />
-      <limit
-        effort="39"
-        velocity="1.3963" />
+      <limit lower="-0.35" upper="0.35" effort="39" velocity="0.87" />
     </joint>
     <link name="${prefix}forearm_link">
@@ -164,5 +160,5 @@
       <axis
         xyz="0 0 1" />
-      <limit lower="-2.66" upper="2.66" effort="39" velocity="1.3963" />
+      <limit lower="0.0" upper="2.66" effort="39" velocity="0.87" />
     </joint>
     <link name="${prefix}spherical_wrist_1_link">
@@ -190,5 +186,5 @@
     <joint
       name="${prefix}joint_5"
-      type="continuous">
+      type="revolute">
       <origin xyz="0 -0.20843 -0.006375" rpy="-1.5708 2.2204E-16 -6.373E-17" />
       <parent
@@ -198,7 +194,5 @@
       <axis
         xyz="0 0 1" />
-      <limit
-        effort="9"
-        velocity="1.2218" />
+      <limit lower="-3.0" upper="3.0" effort="39" velocity="0.87" />
     </joint>
     <link name="${prefix}spherical_wrist_2_link">
@@ -234,5 +228,5 @@
       <axis
         xyz="0 0 1" />
-      <limit lower="-2.23" upper="2.23" effort="9" velocity="1.2218" />
+      <limit lower="0.0" upper="2.23" effort="39" velocity="0.87" />
     </joint>
     <xacro:if value="${vision}">
@@ -286,5 +280,5 @@
     <joint
       name="${prefix}joint_7"
-      type="continuous">
+      type="revolute">
       <origin xyz="0 -0.10593 -0.00017505" rpy="-1.5708 -5.5511E-17 9.6396E-17" />
       <parent
@@ -294,7 +288,5 @@
       <axis
         xyz="0 0 1" />
-      <limit
-        effort="9"
-        velocity="1.2218" />
+      <limit lower="-3.1" upper="3.1" effort="39" velocity="0.87" />
     </joint>
     <link name="${prefix}end_effector_link" />

File: kortex_description/robots/kortex_robot.xacro (robot description, xacro)
@@ -52,5 +52,5 @@
             <joint name="${prefix}tool_frame_joint" type="fixed">
                 <!-- origin xyz="0 0 0" rpy="0 0 0" / -->
-                <origin xyz="-0.41 0 0.02" rpy="0 -1.5707 3.14159" />
+                <origin xyz="-0.41 0 0.02" rpy="1.5707 0 1.5707" />
                 <parent link="${prefix}${last_arm_link}" />
                 <child link="${prefix}tool_frame" />
